File: Pico_STEMMA_HAT/Pico_STEMMA_HAT.kicad_sch (KiCad schematic)
At the start: 55 parts, among them J1 Conn_01x20_Socket, J2 Conn_01x20_Socket, J3 SDCARD_MODULE

Commit message: Change reset pin to be out in the open
Parts:
- added R29: 10k, Resistor_SMD:R_0603_1608Metric, symbol Device:R_US
- added TP1: RESET PIN, TestPoint:TestPoint_THTPad_1.0x1.0mm_Drill0.5mm, symbol Connector:TestPoint
Connections:
- net +3V3: now also R29.1
- net RESET: now reaches TCA9548A1.3 (#RESET)
- net RESET: now also R29.2, TP1.1
- no-connect marks 24 -> 23
Other:
- moved on the sheet: JP1, JP2, JP3, R26, R27, R28

Commit message: Update schematic formatting
Other:
- note added: "Neopixel"
- note added: "RASPBERRY PI PICO HEADER CONNECTIONS"
- note removed: "MQTT STATUS NEOPIXEL"
- note removed: "RASPBERRY PI PICO W HEADER CONNECTIONS"
- moved on the sheet: C1, C10, C2, C3, C4, C5, C6, C7, C8, C9, D1, D2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

Commit message: Update schematic
Other:
- moved on the sheet: C1, C2, C3, C4, C5, C6, C7, C8, R1, R10, R11, R12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
